File: Lab_1_Morris_Lin_ASIC_II.kicad_sch (KiCad schematic)
At the start: 106 parts, among them IC1 74CBTLV3253D,118, IC2 74CBTLV3253D,118, IC3 74CBTLV3253D,118, IC4 74CBTLV3253D,118, IC5 74CBTLV3253D,118, IC6 74CBTLV3253D,118, J10 Conn_01x14, J11 Conn_01x14, J12 VDDPST External, J2 PMOD_A, J3 PMOD_B, J4 VDD_Qn External, J5 VDDRING External, J6 Logic_Analyzer_PMOD_A, J7 Logic_Analyzer_PMOD_B, J8 Conn_01x14, J9 Conn_01x14, Q1 BSS138P, U1 TLV75710PDBV, U2 TLV75710PDBV

Commit message: Changed LED curr limit and PTC Fuse values
Parts:
- F1: value SMDH1206B025TF -> SMDH1206B030TF; Mouser Part Number 603-SMDH1206B025TF -> 603-SMDH1206B030TF
- R1, R2, R3, R39, R4, R7, R9: value 470 -> 120; Mouser Part Number 603-RC1206FR-13470RL -> 71-CRCW1206120RJNEAC
Changed lines of the file:
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@@
 			)
 		)
-		(property "Value" "470"
+		(property "Value" "120"
 			(at 41.91 236.2199 0)
 			(show_name no)
@@
 			)
 		)
-		(property "Mouser Part Number" " 603-RC1206FR-13470RL "
+		(property "Mouser Part Number" " 71-CRCW1206120RJNEAC "
 			(at 39.37 234.95 0)
 			(hide yes)
@@
 			)
 		)
-		(property "Value" "470"
+		(property "Value" "120"
 			(at 67.31 236.2199 0)
 			(show_name no)
@@
 			)
 		)
-		(property "Mouser Part Number" " 603-RC1206FR-13470RL "
+		(property "Mouser Part Number" " 71-CRCW1206120RJNEAC "
 			(at 64.77 234.95 0)
 			(hide yes)
@@
 			)
 		)
-		(property "Value" "SMDH1206B025TF"
+		(property "Value" "SMDH1206B030TF"
 			(at 57.15 21.59 90)
 			(show_name no)
@@
 			)
 		)
-		(property "Mouser Part Number" "603-SMDH1206B025TF "
+		(property "Mouser Part Number" " 603-SMDH1206B030TF "
 			(at 57.15 25.4 90)
 			(hide yes)
@@
 			)
 		)
-		(property "Value" "470"
+		(property "Value" "120"
 			(at 109.22 228.5999 0)
 			(show_name no)
@@
 			)
 		)
-		(property "Mouser Part Number" " 603-RC1206FR-13470RL "
+		(property "Mouser Part Number" " 71-CRCW1206120RJNEAC "
 			(at 106.68 227.33 0)
 			(hide yes)
@@
 			)
 		)
-		(property "Value" "470"
+		(property "Value" "120"
 			(at 118.11 31.7499 0)
 			(show_name no)
@@
 			)
 		)
-		(property "Mouser Part Number" " 603-RC1206FR-13470RL "
+		(property "Mouser Part Number" " 71-CRCW1206120RJNEAC "
 			(at 115.57 30.48 0)
 			(hide yes)
@@
 			)
 		)
-		(property "Value" "470"
+		(property "Value" "120"
 			(at 54.61 236.2199 0)
 			(show_name no)
@@
 			)
 		)
-		(property "Mouser Part Number" " 603-RC1206FR-13470RL "
+		(property "Mouser Part Number" " 71-CRCW1206120RJNEAC "
 			(at 52.07 234.95 0)
 			(hide yes)
@@
 			)
 		)
-		(property "Value" "470"
+		(property "Value" "120"
 			(at 118.11 69.8499 0)
 			(show_name no)
@@
 			)
 		)
-		(property "Mouser Part Number" " 603-RC1206FR-13470RL "
+		(property "Mouser Part Number" " 71-CRCW1206120RJNEAC "
 			(at 115.57 68.58 0)
 			(hide yes)
@@
 			)
 		)
-		(property "Value" "470"
+		(property "Value" "120"
 			(at 29.21 236.2199 0)
 			(show_name no)
@@
 			)
 		)
-		(property "Mouser Part Number" " 603-RC1206FR-13470RL "
+		(property "Mouser Part Number" " 71-CRCW1206120RJNEAC "
 			(at 26.67 234.95 0)
 			(hide yes)
